Commit message: corrected for inertias

File: aquanaute_description/urdf/aquanaute.urdf (robot description, URDF)
Before this commit: robot aquanaute, 5 links, 4 joints
Links:
- added link platform_link, mass 16; collision mesh filename=package://aquanaute_description/models/meshes/Platform.stl; visual mesh filename=package://aquanaute_description/models/meshes/Platform.stl
- link base_link: geometry visual sphere radius=0.001
- link left_hull_link: mass None -> 10.45
- link motor_link: mass None -> 6.6
- link right_hull_link: mass None -> 10.45
- link sensor_frame_link: mass None -> 1.8
Joints:
- added joint platform_base_joint: type fixed, parent base_link, child platform_link, origin xyz=0 0 0 rpy=0 0 0
- joint left_hull_platform_joint: parent base_link -> platform_link
- joint right_hull_platform_joint: parent base_link -> platform_link
