Commit message: spawn correct - flotation incorrect

File: aquanaute_description/urdf/aquanaute_description.urdf.xacro (robot description, xacro)
@@ -1,4 +1,4 @@
 <?xml version="1.0"?>
-<robot name="aquanaute">
+<robot xmlns:xacro="http://ros.org/wiki/xacro" name="aquanaute">
     <material name="blue">
         <color rgba="0 0 0.8 1"/>
@@ -184,5 +184,5 @@
         <mu1>10.0</mu1>
         <mu2>10.0</mu2>
-        <material>Gazebo/Grey</material>
+        <material>Gazebo/Red</material>
     </gazebo>
     <gazebo reference="left_hull_link">
@@ -191,5 +191,5 @@
         <mu1>10.0</mu1>
         <mu2>10.0</mu2>
-        <material>Gazebo/Grey</material>
+        <material>Gazebo/Red</material>
     </gazebo>
     <gazebo reference="motor_link">
@@ -198,5 +198,5 @@
         <mu1>10.0</mu1>
         <mu2>10.0</mu2>
-        <material>Gazebo/Grey</material>
+        <material>Gazebo/Black</material>
     </gazebo>
     <gazebo reference="sensor_frame_link">
@@ -205,31 +205,5 @@
         <mu1>10.0</mu1>
         <mu2>10.0</mu2>
-        <material>Gazebo/Grey</material>
-    </gazebo>
-    <!--
-    <joint name="pitch_joint" type="revolute">
-    	<parent link="roll_M1_link"/>
-    	<child link="pitch_M2_link"/>
-    	<origin xyz="0 0 0" rpy="0 -1.5708 0"/>
-        <limit lower="0" upper="0.44" effort="0.1" velocity="0.005"/>
-        <axis xyz="0 1 0"/>
-	</joint>
-    <joint name="yaw_joint" type="continuous">
-    	<parent link="pitch_M2_link"/>
-    	<child link="yaw_M3_link"/>
-        <origin xyz="0.01 0 0" rpy="0 1.5708 0"/>
-        <limit effort="0.1" velocity="0.01"/>
-        <axis xyz="0 0 1"/>
-	</joint>
-    -->
-    <!-- This is for color and physical properties in Gazebo, color won't work with the material tag in gazebo
-    only for URDF coloring
-    <gazebo reference="roll_M1_link">
-        <kp>1000.0</kp>
-        <kd>10.0</kd>
-        <mu1>10.0</mu1>
-        <mu2>10.0</mu2>
-        <material>Gazebo/Red</material>
-    </gazebo>
-    -->
+        <material>Gazebo/White</material>
+    </gazebo>
 </robot>

File: vrx_gazebo/worlds/ocean.world.xacro (robot description, xacro)
@@ -43,5 +43,4 @@
     <!-- World models  -->
     <xacro:include filename="$(find wave_gazebo)/world_models/ocean_waves/model.xacro"/>
-    <xacro:ocean_waves gain="0.6"/>
   </world>
 </sdf>

File: vrx_gazebo/worlds/xacros/usv_wind_plugin.xacro (robot description, xacro)
@@ -6,5 +6,5 @@
                          mean_vel:=0
                          var_gain:=0
-                         var_time:=1
+                         var_time:=0
                          seed:=''
                          ros_update_rate:=10

File: wave_gazebo/world_models/ocean_waves/model.xacro (robot description, xacro)
@@ -17,77 +17,75 @@
 -->
 <world xmlns:xacro="http://ros.org/wiki/xacro">
-  <xacro:macro name="ocean_waves" params="gain:=0.1 period:=5
-                     direction_x:=1.0 direction_y:=0.0
-                     angle:=0.4">
-  <model name='ocean_waves'>
-    <static>true</static>
-    <plugin name="wavefield_plugin" filename="libWavefieldModelPlugin.so">
-      <static>false</static>
-      <update_rate>30</update_rate>
-      <size>1000 1000</size>
-      <cell_count>50 50</cell_count>
-      <wave>
-				<model>PMS</model>
-        <period>${period}</period>
-        <number>3</number>
-        <scale>1.5</scale>
-      S	<gain>${gain}</gain>
-        <direction>${direction_x} ${direction_y}</direction>
-        <angle>${angle}</angle>
-        <tau>2.0</tau>
-        <amplitude>0.0</amplitude>  <!-- No effect for the PMS model -->
-        <steepness>0.0</steepness>
-      </wave>
-    </plugin>
-    <link name="ocean_waves_link">
-      <visual name="ocean_waves_visual">
-        <plugin name="ocean_waves_visual_plugin" filename="libWavefieldVisualPlugin.so">
-          <enableRtt>true</enableRtt>
-          <rttNoise>0.1</rttNoise>
-          <refractOpacity>0.2</refractOpacity>
-          <reflectOpacity>0.2</reflectOpacity>
-          <wave>
-            <model>PMS</model>
-            <period>${period}</period>
-            <number>3</number>
-            <scale>1.5</scale>
-	    <gain>${gain}</gain>
-            <direction>${direction_x} ${direction_y}</direction>
-            <angle>${angle}</angle>
-            <tau>2.0</tau>
-            <amplitude>0.0</amplitude>  <!-- No effect for the PMS model -->
-            <steepness>0.0</steepness>
-          </wave>
-        </plugin>
-        <geometry>
-          <mesh>
-            <uri>model://ocean_waves/meshes/mesh.dae</uri>
-          </mesh>
-        </geometry>
-        <material>
-          <script>
-            <uri>model://ocean_waves/materials/scripts/waves.material</uri>
-            <name>WaveSim/GerstnerWaves</name>
-          </script>
-        </material>
-        <laser_retro>-1</laser_retro>
-      </visual>
-      <visual name="ocean_waves_below_visual">
-        <pose>0 0 -0.05 0 0 0</pose>  <!-- Offset to prevent rendering conflict -->
-        <geometry>
-          <mesh>
-            <uri>model://ocean_waves/meshes/mesh_below.dae</uri>
-          </mesh>
-        </geometry>
-        <material>
-          <script>
-            <uri>model://ocean_waves/materials/scripts/waves.material</uri>
-            <name>WaveSim/GerstnerWaves</name>
-          </script>
-        </material>
-        <laser_retro>-1</laser_retro>
-      </visual>
-    </link>
-  </model>
+  <xacro:macro name="ocean_waves" params="gain:=0.0 period:=5 direction_x:=1.0 direction_y:=0.0 angle:=0.4">
+    <model name='ocean_waves'>
+      <static>true</static>
+      <plugin name="wavefield_plugin" filename="libWavefieldModelPlugin.so">
+        <static>false</static>
+        <update_rate>30</update_rate>
+        <size>500 500</size>
+        <cell_count>50 50</cell_count>
+        <wave>
+          <model>PMS</model>
+          <period>${period}</period>
+          <number>3</number>
+          <scale>1.5</scale>
+          <gain>${gain}</gain>
+          <direction>${direction_x} ${direction_y}</direction>
+          <angle>${angle}</angle>
+          <tau>2.0</tau>
+          <amplitude>0.0</amplitude>          <!-- No effect for the PMS model -->
+          <steepness>0.0</steepness>
+        </wave>
+      </plugin>
+      <link name="ocean_waves_link">
+        <visual name="ocean_waves_visual">
+          <plugin name="ocean_waves_visual_plugin" filename="libWavefieldVisualPlugin.so">
+            <enableRtt>true</enableRtt>
+            <rttNoise>0.1</rttNoise>
+            <refractOpacity>0.2</refractOpacity>
+            <reflectOpacity>0.2</reflectOpacity>
+            <wave>
+              <model>PMS</model>
+              <period>${period}</period>
+              <number>3</number>
+              <scale>1.5</scale>
+              <gain>${gain}</gain>
+              <direction>${direction_x} ${direction_y}</direction>
+              <angle>${angle}</angle>
+              <tau>2.0</tau>
+              <amplitude>0.0</amplitude>              <!-- No effect for the PMS model -->
+              <steepness>0.0</steepness>
+            </wave>
+          </plugin>
+          <geometry>
+            <mesh>
+              <uri>model://ocean_waves/meshes/mesh.dae</uri>
+            </mesh>
+          </geometry>
+          <material>
+            <script>
+              <uri>model://ocean_waves/materials/scripts/waves.material</uri>
+              <name>WaveSim/GerstnerWaves</name>
+            </script>
+          </material>
+          <laser_retro>-1</laser_retro>
+        </visual>
+        <visual name="ocean_waves_below_visual">
+          <pose>0 0 -0.05 0 0 0</pose>          <!-- Offset to prevent rendering conflict -->
+          <geometry>
+            <mesh>
+              <uri>model://ocean_waves/meshes/mesh_below.dae</uri>
+            </mesh>
+          </geometry>
+          <material>
+            <script>
+              <uri>model://ocean_waves/materials/scripts/waves.material</uri>
+              <name>WaveSim/GerstnerWaves</name>
+            </script>
+          </material>
+          <laser_retro>-1</laser_retro>
+        </visual>
+      </link>
+    </model>
   </xacro:macro>
 </world>

Commit message: spawn of aquanate correct with wind and waves - missing thruster input

File: aquanaute_description/urdf/aquanaute_description.urdf.xacro (robot description, xacro)
@@ -142,5 +142,5 @@
     	<parent link="base_link"/>
     	<child link="platform_link"/>
-    	<origin xyz="0 0 0" rpy="0 0 0"/>
+    	<origin xyz="0 0 0.35" rpy="0 0 0"/>
 	</joint>
     <joint name="right_hull_platform_joint" type="fixed">
@@ -155,10 +155,10 @@
 	</joint>
     <joint name="motor_platform_joint" type="fixed">
-    	<parent link="base_link"/>
+    	<parent link="platform_link"/>
     	<child link="motor_link"/>
     	<origin xyz="-0.91 0.0 -0.09" rpy="0 0 0"/>
 	</joint>
     <joint name="sensor_frame_platform_joint" type="fixed">
-    	<parent link="base_link"/>
+    	<parent link="platform_link"/>
     	<child link="sensor_frame_link"/>
     	<origin xyz="-0.55 0.0 0.0" rpy="0 0 0"/>

File: aquanaute_gazebo/urdf/aquanaute_gazebo.urdf.xacro (robot description, xacro)
@@ -5,5 +5,5 @@
     <xacro:include filename="$(find aquanaute_gazebo)/urdf/macros.xacro" />
     <!-- Defines the base vehicle -->
-    <xacro:include filename="$(find aquanaute_description)/urdf/aquanaute_description.urdf.xacro" />
+    <xacro:include filename="$(find aquanaute_description)/urdf/aquanaute_description.urdf.xacro" name="aquanaute"/>
     <!-- Attach hydrodynamics plugin -->
     <xacro:usv_dynamics_gazebo name="aquanaute_dynamics_plugin"/>

File: aquanaute_gazebo/urdf/dynamics/aquanaute_gazebo_dynamics_plugin.xacro (robot description, xacro)
@@ -10,7 +10,7 @@
         <waterDensity>997.8</waterDensity>
         <!-- Added mass -->
-        <xDotU>0.0</xDotU>
-        <yDotV>0.0</yDotV>
-        <nDotR>0.0</nDotR>
+        <xDotU>10.0</xDotU>
+        <yDotV>10.0</yDotV>
+        <nDotR>25.0</nDotR>
         <!-- Linear and quadratic drag -->
         <xU>51.3</xU>
@@ -25,7 +25,7 @@
         <!-- General dimensions -->
         <!--<boatArea>2.2</boatArea>-->
-        <hullRadius>0.19</hullRadius>
-        <boatWidth>2</boatWidth>
-        <boatLength>3</boatLength>
+        <hullRadius>0.18</hullRadius>
+        <boatWidth>1.8</boatWidth>
+        <boatLength>3.0</boatLength>
         <!-- Length discretization, AKA, "N" -->
         <length_n>10</length_n>

Commit message: added pluggin for ardupilot

File: aquanaute_description/urdf/aquanaute_description.urdf.xacro (robot description, xacro)
@@ -1,4 +1,4 @@
 <?xml version="1.0"?>
-<robot xmlns:xacro="http://ros.org/wiki/xacro">
+<robot xmlns:xacro="http://ros.org/wiki/xacro" name="aquanaute">
     <material name="blue">
         <color rgba="0 0 0.8 1"/>
@@ -8,5 +8,5 @@
     </material>
     <material name="green">
-        <color rgba="0 0.8 0 1"/>
+        <color rgba="0 0.8 0 0.5"/>
     </material>
     <material name="cyan">
@@ -28,5 +28,5 @@
         <color rgba="0 0 0 1"/>
     </material>
-   	<!-- * * * Link Definitions * * * -->
+    <!-- * * * Link Definitions * * * -->
     <link name="base_link">
         <visual>
@@ -118,9 +118,24 @@
         </visual>
     </link>
+    <link name="propeller_link">
+        <collision>
+            <origin xyz="0 0 0" rpy="0 0 0"/>
+            <geometry>
+                <cylinder radius="0.05" length="0.04"/>
+            </geometry>
+        </collision>
+        <visual>
+            <origin rpy="0 0 0" xyz="0 0 0"/>
+            <geometry>
+                <cylinder radius="0.01" length="0.02"/>
+            </geometry>
+            <material name="green"/>
+        </visual>
+    </link>
     <link name="sensor_frame_link">
         <inertial>
             <origin xyz="-0.007 0 0.379" rpy="0 0 0"/>
             <mass value="1.8"/>
-            <inertia ixx="0.308" ixy="0.00" ixz="0.007" iyy="0.297"	iyz="0.00" izz="0.022"/>
+            <inertia ixx="0.308" ixy="0.00" ixz="0.007" iyy="0.297" iyz="0.00" izz="0.022"/>
         </inertial>
         <collision>
@@ -140,28 +155,37 @@
     <!-- * * * Joint Definitions * * * -->
     <joint name="platform_base_joint" type="fixed">
-    	<parent link="base_link"/>
-    	<child link="platform_link"/>
-    	<origin xyz="0 0 0.35" rpy="0 0 0"/>
-	</joint>
+        <parent link="base_link"/>
+        <child link="platform_link"/>
+        <origin xyz="0 0 0.35" rpy="0 0 0"/>
+    </joint>
     <joint name="right_hull_platform_joint" type="fixed">
-    	<parent link="platform_link"/>
-    	<child link="right_hull_link"/>
-    	<origin xyz="-0.05 -0.7 -0.036" rpy="0 0 0"/>
-	</joint>
+        <parent link="platform_link"/>
+        <child link="right_hull_link"/>
+        <origin xyz="-0.05 -0.7 -0.036" rpy="0 0 0"/>
+    </joint>
     <joint name="left_hull_platform_joint" type="fixed">
-    	<parent link="platform_link"/>
-    	<child link="left_hull_link"/>
-    	<origin xyz="-0.05 0.7 -0.036" rpy="0 0 0"/>
-	</joint>
-    <joint name="motor_platform_joint" type="fixed">
-    	<parent link="platform_link"/>
-    	<child link="motor_link"/>
-    	<origin xyz="-0.91 0.0 -0.09" rpy="0 0 0"/>
-	</joint>
+        <parent link="platform_link"/>
+        <child link="left_hull_link"/>
+        <origin xyz="-0.05 0.7 -0.036" rpy="0 0 0"/>
+    </joint>
+    <joint name="motor_platform_joint" type="revolute">
+        <parent link="platform_link"/>
+        <child link="motor_link"/>
+        <origin xyz="-0.91 0.0 -0.09" rpy="0 0 0"/>
+        <axis xyz="0 0 1"/>
+        <limit effort="-1" velocity="-1" lower="-0.9" upper="0.9"/>
+    </joint>
+    <joint name="propeller_motor_joint" type="revolute">
+        <parent link="motor_link"/>
+        <child link="propeller_link"/>
+        <origin xyz="-0.28 0 -0.42" rpy="0 1.57 0"/>
+        <axis xyz="0 0 1"/>
+        <limit effort="-1" velocity="-1" lower="-1e+12" upper="1e+12"/>
+    </joint>
     <joint name="sensor_frame_platform_joint" type="fixed">
-    	<parent link="platform_link"/>
-    	<child link="sensor_frame_link"/>
-    	<origin xyz="-0.55 0.0 0.0" rpy="0 0 0"/>
-	</joint>
+        <parent link="platform_link"/>
+        <child link="sensor_frame_link"/>
+        <origin xyz="-0.55 0.0 0.0" rpy="0 0 0"/>
+    </joint>
     <!-- * * * GAZEBO Definitions * * * -->
     <gazebo reference="base_link">
@@ -207,3 +231,46 @@
         <material>Gazebo/White</material>
     </gazebo>
+    <!-- * * * GAZEBO Plugins * * * -->
+    <plugin name="ardupilot_plugin" filename="libArduPilotPlugin.so">
+        <fdm_addr>127.0.0.1</fdm_addr>
+        <fdm_port_in>9002</fdm_port_in>
+        <fdm_port_out>9003</fdm_port_out>
+        <modelXYZToAirplaneXForwardZDown>0 0 0 3.141593 0 0</modelXYZToAirplaneXForwardZDown>
+        <gazeboXYZToNED>0 0 0 3.141593 0 0</gazeboXYZToNED>
+        <!--<imuName></imuName>-->
+        <connectionTimeoutMaxCount>5</connectionTimeoutMaxCount>
+        <!--
+          incoming control command [0, 1]
+          so offset it by 0 to get [0, 1]
+          and divide max target by 1.
+          offset = 0
+          multiplier = 838 max rpm / 1 = 838
+        -->
+        <control channel="0">
+            <multiplier>1</multiplier>
+            <offset>-0.5</offset>
+            <type>RIC</type>
+            <p_gain>1</p_gain>
+            <i_gain>0</i_gain>
+            <d_gain>0</d_gain>
+            <i_max>0</i_max>
+            <i_min>0</i_min>
+            <cmd_max>1</cmd_max>
+            <cmd_min>-1</cmd_min>
+            <jointName>aquanaute::motor_platform_joint</jointName>
+        </control>
+        <control channel="1">
+            <multiplier>1</multiplier>
+            <offset>-0.5</offset>
+            <type>THOMAS</type>
+            <p_gain>1</p_gain>
+            <i_gain>0</i_gain>
+            <d_gain>0</d_gain>
+            <i_max>0</i_max>
+            <i_min>0</i_min>
+            <cmd_max>1</cmd_max>
+            <cmd_min>-1</cmd_min>
+            <jointName>aquanaute::propeller_motor_joint</jointName>
+        </control>
+    </plugin>
 </robot>
