Commit message: added imu for plugin - missing fix for error with 2 joints

File: aquanaute_description/urdf/aquanaute_description.urdf.xacro (robot description, xacro)
@@ -128,7 +128,7 @@
             <origin rpy="0 0 0" xyz="0 0 0"/>
             <geometry>
-                <cylinder radius="0.01" length="0.02"/>
-            </geometry>
-            <material name="green"/>
+                <cylinder radius="0.04" length="0.05"/>
+            </geometry>
+            <material name="black"/>
         </visual>
     </link>
@@ -149,4 +149,13 @@
             <geometry>
                 <mesh filename="package://aquanaute_description/models/meshes/sensor_frame.stl"/>
+            </geometry>
+            <material name="cyan"/>
+        </visual>
+    </link>
+    <link name="imu_link">
+        <visual>
+            <origin rpy="0.0 0 0" xyz="0 0 0"/>
+            <geometry>
+                <cylinder radius="0.04" length="0.05"/>
             </geometry>
             <material name="cyan"/>
@@ -176,10 +185,10 @@
         <limit effort="-1" velocity="-1" lower="-0.9" upper="0.9"/>
     </joint>
-    <joint name="propeller_motor_joint" type="revolute">
+    <joint name="propeller_motor_joint" type="fixed">
         <parent link="motor_link"/>
         <child link="propeller_link"/>
-        <origin xyz="-0.28 0 -0.42" rpy="0 1.57 0"/>
+        <origin xyz="-0.5 0 0.42" rpy="0 1.57 0"/>
         <axis xyz="0 0 1"/>
-        <limit effort="-1" velocity="-1" lower="-1e+12" upper="1e+12"/>
+        <limit effort="-1" velocity="-1" lower="-1e+16" upper="1e+16"/>
     </joint>
     <joint name="sensor_frame_platform_joint" type="fixed">
@@ -188,89 +197,8 @@
         <origin xyz="-0.55 0.0 0.0" rpy="0 0 0"/>
     </joint>
-    <!-- * * * GAZEBO Definitions * * * -->
-    <gazebo reference="base_link">
-        <kp>100000.0</kp>
-        <kd>100000.0</kd>
-        <mu1>10.0</mu1>
-        <mu2>10.0</mu2>
-        <material>Gazebo/Grey</material>
-    </gazebo>
-    <gazebo reference="platform_link">
-        <kp>100000.0</kp>
-        <kd>100000.0</kd>
-        <mu1>10.0</mu1>
-        <mu2>10.0</mu2>
-        <material>Gazebo/Grey</material>
-    </gazebo>
-    <gazebo reference="right_hull_link">
-        <kp>100000.0</kp>
-        <kd>100000.0</kd>
-        <mu1>10.0</mu1>
-        <mu2>10.0</mu2>
-        <material>Gazebo/Red</material>
-    </gazebo>
-    <gazebo reference="left_hull_link">
-        <kp>100000.0</kp>
-        <kd>100000.0</kd>
-        <mu1>10.0</mu1>
-        <mu2>10.0</mu2>
-        <material>Gazebo/Red</material>
-    </gazebo>
-    <gazebo reference="motor_link">
-        <kp>100000.0</kp>
-        <kd>100000.0</kd>
-        <mu1>10.0</mu1>
-        <mu2>10.0</mu2>
-        <material>Gazebo/Black</material>
-    </gazebo>
-    <gazebo reference="sensor_frame_link">
-        <kp>100000.0</kp>
-        <kd>100000.0</kd>
-        <mu1>10.0</mu1>
-        <mu2>10.0</mu2>
-        <material>Gazebo/White</material>
-    </gazebo>
-    <!-- * * * GAZEBO Plugins * * * -->
-    <plugin name="ardupilot_plugin" filename="libArduPilotPlugin.so">
-        <fdm_addr>127.0.0.1</fdm_addr>
-        <fdm_port_in>9002</fdm_port_in>
-        <fdm_port_out>9003</fdm_port_out>
-        <modelXYZToAirplaneXForwardZDown>0 0 0 3.141593 0 0</modelXYZToAirplaneXForwardZDown>
-        <gazeboXYZToNED>0 0 0 3.141593 0 0</gazeboXYZToNED>
-        <!--<imuName></imuName>-->
-        <connectionTimeoutMaxCount>5</connectionTimeoutMaxCount>
-        <!--
-          incoming control command [0, 1]
-          so offset it by 0 to get [0, 1]
-          and divide max target by 1.
-          offset = 0
-          multiplier = 838 max rpm / 1 = 838
-        -->
-        <control channel="0">
-            <multiplier>1</multiplier>
-            <offset>-0.5</offset>
-            <type>RIC</type>
-            <p_gain>1</p_gain>
-            <i_gain>0</i_gain>
-            <d_gain>0</d_gain>
-            <i_max>0</i_max>
-            <i_min>0</i_min>
-            <cmd_max>1</cmd_max>
-            <cmd_min>-1</cmd_min>
-            <jointName>aquanaute::motor_platform_joint</jointName>
-        </control>
-        <control channel="1">
-            <multiplier>1</multiplier>
-            <offset>-0.5</offset>
-            <type>THOMAS</type>
-            <p_gain>1</p_gain>
-            <i_gain>0</i_gain>
-            <d_gain>0</d_gain>
-            <i_max>0</i_max>
-            <i_min>0</i_min>
-            <cmd_max>1</cmd_max>
-            <cmd_min>-1</cmd_min>
-            <jointName>aquanaute::propeller_motor_joint</jointName>
-        </control>
-    </plugin>
+    <joint name="imu_platform_joint" type="fixed">
+        <parent link="platform_link"/>
+        <child link="imu_link"/>
+        <origin xyz="0 0 0.1" rpy="0 0 0"/>
+    </joint>
 </robot>

File: aquanaute_gazebo/urdf/aquanaute_gazebo.urdf.xacro (robot description, xacro)
@@ -2,9 +2,113 @@
 <!-- Basic WAM-V with gazebo plugins for dynamics -->
 <robot xmlns:xacro="http://ros.org/wiki/xacro">
-    <!-- Include macros for dynamics plugins -->
-    <xacro:include filename="$(find aquanaute_gazebo)/urdf/macros.xacro" />
+    <!-- Include macros for dynamics plugins
+    <xacro:include filename="$(find aquanaute_gazebo)/urdf/macros.xacro" /> -->
     <!-- Defines the base vehicle -->
     <xacro:include filename="$(find aquanaute_description)/urdf/aquanaute_description.urdf.xacro"/>
-    <!-- Attach hydrodynamics plugin -->
-    <xacro:usv_dynamics_gazebo name="aquanaute_dynamics_plugin"/>
+    <!-- Defines the sim plugins-->
+    <gazebo reference="base_link">
+        <kp>100000.0</kp>
+        <kd>100000.0</kd>
+        <mu1>10.0</mu1>
+        <mu2>10.0</mu2>
+        <material>Gazebo/Grey</material>
+    </gazebo>
+    <gazebo reference="platform_link">
+        <kp>100000.0</kp>
+        <kd>100000.0</kd>
+        <mu1>10.0</mu1>
+        <mu2>10.0</mu2>
+        <material>Gazebo/Grey</material>
+    </gazebo>
+    <gazebo reference="right_hull_link">
+        <kp>100000.0</kp>
+        <kd>100000.0</kd>
+        <mu1>10.0</mu1>
+        <mu2>10.0</mu2>
+        <material>Gazebo/Red</material>
+    </gazebo>
+    <gazebo reference="left_hull_link">
+        <kp>100000.0</kp>
+        <kd>100000.0</kd>
+        <mu1>10.0</mu1>
+        <mu2>10.0</mu2>
+        <material>Gazebo/Red</material>
+    </gazebo>
+    <gazebo reference="motor_link">
+        <kp>100000.0</kp>
+        <kd>100000.0</kd>
+        <mu1>10.0</mu1>
+        <mu2>10.0</mu2>
+        <material>Gazebo/Black</material>
+    </gazebo>
+    <gazebo reference="propeller_link">
+        <kp>100000.0</kp>
+        <kd>100000.0</kd>
+        <mu1>10.0</mu1>
+        <mu2>10.0</mu2>
+        <material>Gazebo/Black</material>
+    </gazebo>
+    <gazebo reference="sensor_frame_link">
+        <kp>100000.0</kp>
+        <kd>100000.0</kd>
+        <mu1>10.0</mu1>
+        <mu2>10.0</mu2>
+        <material>Gazebo/White</material>
+    </gazebo>
+    <gazebo>
+        <link name="imu_link">
+            <sensor name="imu_sensor" type="imu">
+                <pose>0 0 0 3.141593 0 0</pose>
+                <always_on>1</always_on>
+                <update_rate>1000.0</update_rate>
+            </sensor>
+        </link>
+    </gazebo>
+    <!-- * * * GAZEBO Plugins * * * -->
+    <gazebo>
+        <plugin name="ardupilot_plugin" filename="libArduPilotPlugin.so">
+            <fdm_addr>127.0.0.1</fdm_addr>
+            <fdm_port_in>9002</fdm_port_in>
+            <fdm_port_out>9003</fdm_port_out>
+            <modelXYZToAirplaneXForwardZDown>0 0 0 3.141593 0 0</modelXYZToAirplaneXForwardZDown>
+            <gazeboXYZToNED>0 0 0 3.141593 0 0</gazeboXYZToNED>
+            <imuName>imu_sensor</imuName>
+            <connectionTimeoutMaxCount>5</connectionTimeoutMaxCount>
+            <!--
+            incoming control command [0, 1]
+            so offset it by 0 to get [0, 1]
+            and divide max target by 1.
+            offset = 0
+            multiplier = 838 max rpm / 1 = 838
+            -->
+            <control channel="0">
+                <multiplier>1</multiplier>
+                <offset>-0.5</offset>
+                <type>POSITION</type>
+                <p_gain>1</p_gain>
+                <i_gain>0</i_gain>
+                <d_gain>0</d_gain>
+                <i_max>0</i_max>
+                <i_min>0</i_min>
+                <cmd_max>1</cmd_max>
+                <cmd_min>-1</cmd_min>
+                <jointName>aquanaute::motor_platform_joint</jointName>
+            </control>
+            <control channel="1">
+                <multiplier>1</multiplier>
+                <offset>-0.5</offset>
+                <type>VELOCITY</type>
+                <p_gain>1</p_gain>
+                <i_gain>0</i_gain>
+                <d_gain>0</d_gain>
+                <i_max>0</i_max>
+                <i_min>0</i_min>
+                <cmd_max>1</cmd_max>
+                <cmd_min>-1</cmd_min>
+                <jointName>aquanaute::propeller_motor_joint</jointName>
+            </control>
+        </plugin>
+    </gazebo>
+    <!-- Attach hydrodynamics plugin
+    <xacro:usv_dynamics_gazebo name="aquanaute_dynamics_plugin"/> -->
 </robot>

Commit message: fixed plugin - error in topic advertisements

File: aquanaute_description/urdf/aquanaute_description.urdf.xacro (robot description, xacro)
@@ -115,20 +115,25 @@
                 <mesh filename="package://aquanaute_description/models/meshes/Motor.stl"/>
             </geometry>
-            <material name="purple"/>
+            <material name="black"/>
         </visual>
     </link>
     <link name="propeller_link">
-        <collision>
-            <origin xyz="0 0 0" rpy="0 0 0"/>
-            <geometry>
-                <cylinder radius="0.05" length="0.04"/>
-            </geometry>
-        </collision>
-        <visual>
-            <origin rpy="0 0 0" xyz="0 0 0"/>
-            <geometry>
-                <cylinder radius="0.04" length="0.05"/>
-            </geometry>
-            <material name="black"/>
+        <inertial>
+            <origin xyz="-0.034 0 0" rpy="0 0 0"/>
+            <mass value="0.233"/>
+            <inertia ixx="1.441e-04" ixy="4.406e-09" ixz="0.00" iyy="1.760e-04"	iyz="2.373e-06" izz="1.961e-04"/>
+        </inertial>
+        <collision>
+            <origin xyz="0 0 0" rpy="0 0 0"/>
+            <geometry>
+                <mesh filename="package://aquanaute_description/models/meshes/Propeller.stl"/>
+            </geometry>
+        </collision>
+        <visual>
+            <origin rpy="0.0 0 0" xyz="0 0 0"/>
+            <geometry>
+                <mesh filename="package://aquanaute_description/models/meshes/Propeller.stl"/>
+            </geometry>
+            <material name="blue"/>
         </visual>
     </link>
@@ -150,5 +155,5 @@
                 <mesh filename="package://aquanaute_description/models/meshes/sensor_frame.stl"/>
             </geometry>
-            <material name="cyan"/>
+            <material name="white"/>
         </visual>
     </link>
@@ -183,12 +188,12 @@
         <origin xyz="-0.91 0.0 -0.09" rpy="0 0 0"/>
         <axis xyz="0 0 1"/>
-        <limit effort="-1" velocity="-1" lower="-0.9" upper="0.9"/>
-    </joint>
-    <joint name="propeller_motor_joint" type="fixed">
+        <limit effort="1" velocity="1" lower="-0.9" upper="0.9"/>
+    </joint>
+    <joint name="propeller_motor_joint" type="revolute">
         <parent link="motor_link"/>
         <child link="propeller_link"/>
-        <origin xyz="-0.5 0 0.42" rpy="0 1.57 0"/>
-        <axis xyz="0 0 1"/>
-        <limit effort="-1" velocity="-1" lower="-1e+16" upper="1e+16"/>
+        <origin xyz="-0.265 0 -0.42" rpy="0 0 0"/>
+        <axis xyz="1 0 0"/>
+        <limit effort="1" velocity="1" lower="-1e+16" upper="1e+16"/>
     </joint>
     <joint name="sensor_frame_platform_joint" type="fixed">
@@ -200,5 +205,5 @@
         <parent link="platform_link"/>
         <child link="imu_link"/>
-        <origin xyz="0 0 0.1" rpy="0 0 0"/>
+        <origin xyz="0 0 0.02" rpy="0 0 0"/>
     </joint>
 </robot>

File: aquanaute_gazebo/urdf/aquanaute_gazebo.urdf.xacro (robot description, xacro)
@@ -2,9 +2,12 @@
 <!-- Basic WAM-V with gazebo plugins for dynamics -->
 <robot xmlns:xacro="http://ros.org/wiki/xacro">
-    <!-- Include macros for dynamics plugins
-    <xacro:include filename="$(find aquanaute_gazebo)/urdf/macros.xacro" /> -->
+    <xacro:arg name="testing" default="false" />
+    <!-- Include macros for dynamics plugins -->
+    <xacro:unless value="$(arg testing)">
+        <xacro:include filename="$(find aquanaute_gazebo)/urdf/macros.xacro" />
+    </xacro:unless>
     <!-- Defines the base vehicle -->
     <xacro:include filename="$(find aquanaute_description)/urdf/aquanaute_description.urdf.xacro"/>
-    <!-- Defines the sim plugins-->
+    <!--Gazebo References-->
     <gazebo reference="base_link">
         <kp>100000.0</kp>
@@ -43,9 +46,9 @@
     </gazebo>
     <gazebo reference="propeller_link">
-        <kp>100000.0</kp>
-        <kd>100000.0</kd>
-        <mu1>10.0</mu1>
-        <mu2>10.0</mu2>
-        <material>Gazebo/Black</material>
+        <kp>1.0</kp>
+        <kd>1.0</kd>
+        <mu1>1.0</mu1>
+        <mu2>1.0</mu2>
+        <material>Gazebo/Blue</material>
     </gazebo>
     <gazebo reference="sensor_frame_link">
@@ -56,12 +59,11 @@
         <material>Gazebo/White</material>
     </gazebo>
-    <gazebo>
-        <link name="imu_link">
-            <sensor name="imu_sensor" type="imu">
-                <pose>0 0 0 3.141593 0 0</pose>
-                <always_on>1</always_on>
-                <update_rate>1000.0</update_rate>
-            </sensor>
-        </link>
+    <gazebo reference="imu_link">
+        <sensor name="imu_sensor" type="imu">
+            <pose>0 0 0 3.141593 0 0</pose>
+            <always_on>1</always_on>
+            <update_rate>1000.0</update_rate>
+        </sensor>
+        <material>Gazebo/Yellow</material>
     </gazebo>
     <!-- * * * GAZEBO Plugins * * * -->
@@ -96,7 +98,6 @@
             </control>
             <control channel="1">
-                <multiplier>1</multiplier>
+                <type>VELOCITY</type>
                 <offset>-0.5</offset>
-                <type>VELOCITY</type>
                 <p_gain>1</p_gain>
                 <i_gain>0</i_gain>
@@ -104,11 +105,14 @@
                 <i_max>0</i_max>
                 <i_min>0</i_min>
-                <cmd_max>1</cmd_max>
-                <cmd_min>-1</cmd_min>
+                <cmd_max>10</cmd_max>
+                <cmd_min>-10</cmd_min>
                 <jointName>aquanaute::propeller_motor_joint</jointName>
+                <multiplier>70</multiplier>
             </control>
         </plugin>
     </gazebo>
-    <!-- Attach hydrodynamics plugin
-    <xacro:usv_dynamics_gazebo name="aquanaute_dynamics_plugin"/> -->
+    <!-- Attach hydrodynamics plugin -->
+    <xacro:unless value="$(arg testing)">
+        <xacro:usv_dynamics_gazebo name="aquanaute_dynamics_plugin"/>
+    </xacro:unless>
 </robot>

Commit message: general order and small fixes - missing fix for ardupilot gazebo error where motors turn without control

File: aquanaute_description/urdf/aquanaute_description.urdf.xacro (robot description, xacro)
@@ -188,5 +188,6 @@
         <origin xyz="-0.91 0.0 -0.09" rpy="0 0 0"/>
         <axis xyz="0 0 1"/>
-        <limit effort="1" velocity="1" lower="-0.9" upper="0.9"/>
+        <limit effort="-1" velocity="-1" lower="-0.9" upper="0.9"/>
+        <dynamics damping="0.0000001"/>
     </joint>
     <joint name="propeller_motor_joint" type="revolute">
@@ -195,5 +196,6 @@
         <origin xyz="-0.265 0 -0.42" rpy="0 0 0"/>
         <axis xyz="1 0 0"/>
-        <limit effort="1" velocity="1" lower="-1e+16" upper="1e+16"/>
+        <limit effort="-1" velocity="-1" lower="-1e+16" upper="1e+16"/>
+        <dynamics damping="0.0000001"/>
     </joint>
     <joint name="sensor_frame_platform_joint" type="fixed">

File: aquanaute_gazebo/urdf/aquanaute_gazebo.urdf.xacro (robot description, xacro)
@@ -39,15 +39,7 @@
     </gazebo>
     <gazebo reference="motor_link">
-        <kp>100000.0</kp>
-        <kd>100000.0</kd>
-        <mu1>10.0</mu1>
-        <mu2>10.0</mu2>
         <material>Gazebo/Black</material>
     </gazebo>
     <gazebo reference="propeller_link">
-        <kp>1.0</kp>
-        <kd>1.0</kd>
-        <mu1>1.0</mu1>
-        <mu2>1.0</mu2>
         <material>Gazebo/Blue</material>
     </gazebo>
@@ -77,37 +69,18 @@
             <imuName>imu_sensor</imuName>
             <connectionTimeoutMaxCount>5</connectionTimeoutMaxCount>
-            <!--
-            incoming control command [0, 1]
-            so offset it by 0 to get [0, 1]
-            and divide max target by 1.
-            offset = 0
-            multiplier = 838 max rpm / 1 = 838
-            -->
             <control channel="0">
+                <type>POSITION</type>
                 <multiplier>1</multiplier>
-                <offset>-0.5</offset>
-                <type>POSITION</type>
-                <p_gain>1</p_gain>
-                <i_gain>0</i_gain>
-                <d_gain>0</d_gain>
-                <i_max>0</i_max>
-                <i_min>0</i_min>
-                <cmd_max>1</cmd_max>
-                <cmd_min>-1</cmd_min>
+                <offset>0</offset>
                 <jointName>aquanaute::motor_platform_joint</jointName>
             </control>
-            <control channel="1">
+            <control channel="0">
                 <type>VELOCITY</type>
-                <offset>-0.5</offset>
-                <p_gain>1</p_gain>
-                <i_gain>0</i_gain>
-                <d_gain>0</d_gain>
-                <i_max>0</i_max>
-                <i_min>0</i_min>
-                <cmd_max>10</cmd_max>
-                <cmd_min>-10</cmd_min>
+                <multiplier>1</multiplier>
+                <offset>0</offset>
                 <jointName>aquanaute::propeller_motor_joint</jointName>
-                <multiplier>70</multiplier>
             </control>
+<!--
+-->
         </plugin>
     </gazebo>

File: aquanaute_gazebo/urdf/dynamics/aquanaute_gazebo_dynamics_plugin.xacro (robot description, xacro)
@@ -10,7 +10,7 @@
         <waterDensity>997.8</waterDensity>
         <!-- Added mass -->
-        <xDotU>10.0</xDotU>
-        <yDotV>10.0</yDotV>
-        <nDotR>25.0</nDotR>
+        <xDotU>0.0</xDotU>
+        <yDotV>0.0</yDotV>
+        <nDotR>0.0</nDotR>
         <!-- Linear and quadratic drag -->
         <xU>51.3</xU>
@@ -29,5 +29,5 @@
         <boatLength>3.0</boatLength>
         <!-- Length discretization, AKA, "N" -->
-        <length_n>10</length_n>
+        <length_n>2</length_n>
         <!-- Wave model -->
         <wave_model>ocean_waves</wave_model>
