Commit message: fixed inertia, and made boat an assambly instead of different parts

File: aquanaute_description/urdf/aquanaute_description.urdf.xacro (robot description, xacro)
@@ -31,5 +31,5 @@
     <link name="base_link">
         <visual>
-            <origin rpy="0.0 0 0" xyz="0 0 0"/>
+            <origin rpy="0 0 0" xyz="0 0 0"/>
             <geometry>
                 <sphere radius="0.001"/>
@@ -38,62 +38,22 @@
         </visual>
     </link>
-    <link name="platform_link">
+    <link name="boat_link">
         <inertial>
-            <origin xyz="-0.024 0 -0007" rpy="0 0 0"/>
-            <mass value="16"/>
-            <inertia ixx="4.206" ixy="0.0" ixz="-0.031" iyy="4.588" iyz="0.0" izz="8.785"/>
+            <origin xyz="0 0 0" rpy="0 0 0"/>
+            <mass value="38.718"/>
+            <inertia ixx="16.283" ixy="0.008" ixz="0.458" iyy="19.728" iyz="0.0" izz="33.013"/>
         </inertial>
         <collision>
             <origin xyz="0 0 0" rpy="0 0 0"/>
             <geometry>
-                <mesh filename="package://aquanaute_description/models/meshes/Platform.stl"/>
+                <mesh filename="package://aquanaute_description/models/meshes/Assambly_aquanaute.stl"/>
             </geometry>
         </collision>
         <visual>
-            <origin rpy="0.0 0 0" xyz="0 0 0"/>
+            <origin rpy="0 0 0" xyz="0 0 0"/>
             <geometry>
-                <mesh filename="package://aquanaute_description/models/meshes/Platform.stl"/>
+                <mesh filename="package://aquanaute_description/models/meshes/Assambly_aquanaute.stl"/>
             </geometry>
-            <material name="yellow"/>
-        </visual>
-    </link>
-    <link name="right_hull_link">
-        <inertial>
-            <origin xyz="-0.124 0 -0.168" rpy="0 0 0"/>
-            <mass value="10.45"/>
-            <inertia ixx="0.244" ixy="3.346" ixz="0.009" iyy="4.974" iyz="-8.274" izz="4.965"/>
-        </inertial>
-        <collision>
-            <origin xyz="0 0 0" rpy="0 0 0"/>
-            <geometry>
-                <mesh filename="package://aquanaute_description/models/meshes/Hull.stl"/>
-            </geometry>
-        </collision>
-        <visual>
-            <origin rpy="0.0 0 0" xyz="0 0 0"/>
-            <geometry>
-                <mesh filename="package://aquanaute_description/models/meshes/Hull.stl"/>
-            </geometry>
-            <material name="red"/>
-        </visual>
-    </link>
-    <link name="left_hull_link">
-        <inertial>
-            <origin xyz="-0.124 0 -0.168" rpy="0 0 0"/>
-            <mass value="10.45"/>
-            <inertia ixx="0.244" ixy="3.346" ixz="0.009" iyy="4.974" iyz="-8.274" izz="4.965"/>
-        </inertial>
-        <collision>
-            <origin xyz="0 0 0" rpy="0 0 0"/>
-            <geometry>
-                <mesh filename="package://aquanaute_description/models/meshes/Hull.stl"/>
-            </geometry>
-        </collision>
-        <visual>
-            <origin rpy="0.0 0 0" xyz="0 0 0"/>
-            <geometry>
-                <mesh filename="package://aquanaute_description/models/meshes/Hull.stl"/>
-            </geometry>
-            <material name="red"/>
+            <material name="gray"/>
         </visual>
     </link>
@@ -111,9 +71,9 @@
         </collision>
         <visual>
-            <origin rpy="0.0 0 0" xyz="0 0 0"/>
+            <origin rpy="0 0 0" xyz="0 0 0"/>
             <geometry>
                 <mesh filename="package://aquanaute_description/models/meshes/Motor.stl"/>
             </geometry>
-            <material name="black"/>
+            <material name="purple"/>
         </visual>
     </link>
@@ -122,5 +82,6 @@
             <origin xyz="-0.034 0 0" rpy="0 0 0"/>
             <mass value="0.233"/>
-            <inertia ixx="1.441e-04" ixy="4.406e-09" ixz="0.00" iyy="1.760e-04"	iyz="2.373e-06" izz="1.961e-04"/>
+            <!--<inertia ixx="1.441e-04" ixy="4.406e-09" ixz="0.00" iyy="1.760e-04"	iyz="2.373e-06" izz="1.961e-04"/>-->
+            <inertia ixx="0.00" ixy="0.00" ixz="0.00" iyy="0.00" iyz="0.00" izz="0.00"/>
         </inertial>
         <collision>
@@ -131,5 +92,5 @@
         </collision>
         <visual>
-            <origin rpy="0.0 0 0" xyz="0 0 0"/>
+            <origin rpy="0 0 0" xyz="0 0 0"/>
             <geometry>
                 <mesh filename="package://aquanaute_description/models/meshes/Propeller.stl"/>
@@ -138,27 +99,7 @@
         </visual>
     </link>
-    <link name="sensor_frame_link">
-        <inertial>
-            <origin xyz="-0.007 0 0.379" rpy="0 0 0"/>
-            <mass value="1.8"/>
-            <inertia ixx="0.308" ixy="0.00" ixz="0.007" iyy="0.297" iyz="0.00" izz="0.022"/>
-        </inertial>
-        <collision>
-            <origin xyz="0 0 0" rpy="0 0 0"/>
-            <geometry>
-                <mesh filename="package://aquanaute_description/models/meshes/sensor_frame.stl"/>
-            </geometry>
-        </collision>
-        <visual>
-            <origin rpy="0.0 0 0" xyz="0 0 0"/>
-            <geometry>
-                <mesh filename="package://aquanaute_description/models/meshes/sensor_frame.stl"/>
-            </geometry>
-            <material name="white"/>
-        </visual>
-    </link>
     <link name="imu_link">
         <visual>
-            <origin rpy="0.0 0 0" xyz="0 0 0"/>
+            <origin rpy="0 0 0" xyz="0 0 0"/>
             <geometry>
                 <cylinder radius="0.04" length="0.05"/>
@@ -168,21 +109,11 @@
     </link>
     <!-- * * * Joint Definitions * * * -->
-    <joint name="platform_base_joint" type="fixed">
+    <joint name="boat_base_joint" type="fixed">
         <parent link="base_link"/>
-        <child link="platform_link"/>
-        <origin xyz="0 0 0.35" rpy="0 0 0"/>
+        <child link="boat_link"/>
+        <origin xyz="0 0 0.25" rpy="0 0 0"/>
     </joint>
-    <joint name="right_hull_platform_joint" type="fixed">
-        <parent link="platform_link"/>
-        <child link="right_hull_link"/>
-        <origin xyz="-0.05 -0.7 -0.036" rpy="0 0 0"/>
-    </joint>
-    <joint name="left_hull_platform_joint" type="fixed">
-        <parent link="platform_link"/>
-        <child link="left_hull_link"/>
-        <origin xyz="-0.05 0.7 -0.036" rpy="0 0 0"/>
-    </joint>
-    <joint name="motor_platform_joint" type="revolute">
-        <parent link="platform_link"/>
+    <joint name="motor_boat_joint" type="revolute">
+        <parent link="boat_link"/>
         <child link="motor_link"/>
         <origin xyz="-0.91 0.0 -0.09" rpy="0 0 0"/>
@@ -199,13 +130,8 @@
         <dynamics damping="0.0000001"/>
     </joint>
-    <joint name="sensor_frame_platform_joint" type="fixed">
-        <parent link="platform_link"/>
-        <child link="sensor_frame_link"/>
-        <origin xyz="-0.55 0.0 0.0" rpy="0 0 0"/>
-    </joint>
-    <joint name="imu_platform_joint" type="fixed">
-        <parent link="platform_link"/>
+    <joint name="imu_boat_joint" type="fixed">
+        <parent link="boat_link"/>
         <child link="imu_link"/>
-        <origin xyz="0 0 0.02" rpy="0 0 0"/>
+        <origin xyz="0 0 0.04" rpy="0 0 0"/>
     </joint>
 </robot>

File: aquanaute_gazebo/urdf/aquanaute_gazebo.urdf.xacro (robot description, xacro)
@@ -11,4 +11,7 @@
     <!--Gazebo References-->
     <gazebo reference="base_link">
+        <material>Gazebo/Grey</material>
+    </gazebo>
+    <gazebo reference="boat_link">
         <kp>100000.0</kp>
         <kd>100000.0</kd>
@@ -17,36 +20,8 @@
         <material>Gazebo/Grey</material>
     </gazebo>
-    <gazebo reference="platform_link">
-        <kp>100000.0</kp>
-        <kd>100000.0</kd>
-        <mu1>10.0</mu1>
-        <mu2>10.0</mu2>
-        <material>Gazebo/Grey</material>
-    </gazebo>
-    <gazebo reference="right_hull_link">
-        <kp>100000.0</kp>
-        <kd>100000.0</kd>
-        <mu1>10.0</mu1>
-        <mu2>10.0</mu2>
-        <material>Gazebo/Red</material>
-    </gazebo>
-    <gazebo reference="left_hull_link">
-        <kp>100000.0</kp>
-        <kd>100000.0</kd>
-        <mu1>10.0</mu1>
-        <mu2>10.0</mu2>
-        <material>Gazebo/Red</material>
-    </gazebo>
     <gazebo reference="motor_link">
-        <material>Gazebo/Black</material>
+        <material>Gazebo/Blue</material>
     </gazebo>
     <gazebo reference="propeller_link">
-        <material>Gazebo/Blue</material>
-    </gazebo>
-    <gazebo reference="sensor_frame_link">
-        <kp>100000.0</kp>
-        <kd>100000.0</kd>
-        <mu1>10.0</mu1>
-        <mu2>10.0</mu2>
         <material>Gazebo/White</material>
     </gazebo>
@@ -57,5 +32,5 @@
             <update_rate>1000.0</update_rate>
         </sensor>
-        <material>Gazebo/Yellow</material>
+        <material>Gazebo/White</material>
     </gazebo>
     <!-- * * * GAZEBO Plugins * * * -->
@@ -80,5 +55,5 @@
                 <cmd_max>3.5</cmd_max>
                 <cmd_min>-3.5</cmd_min>
-                <jointName>aquanaute::motor_platform_joint</jointName>
+                <jointName>aquanaute::motor_boat_joint</jointName>
             </control>
             <control channel="2">

File: aquanaute_gazebo/urdf/dynamics/aquanaute_gazebo_dynamics_plugin.xacro (robot description, xacro)
@@ -25,9 +25,9 @@
         <!-- General dimensions -->
         <!--<boatArea>2.2</boatArea>-->
-        <hullRadius>0.18</hullRadius>
+        <hullRadius>0.19</hullRadius>
         <boatWidth>1.8</boatWidth>
-        <boatLength>3.0</boatLength>
+        <boatLength>3.2</boatLength>
         <!-- Length discretization, AKA, "N" -->
-        <length_n>2</length_n>
+        <length_n>10</length_n>
         <!-- Wave model -->
         <wave_model>ocean_waves</wave_model>

Commit message: corrections

File: aquanaute_description/urdf/aquanaute_description.urdf.xacro (robot description, xacro)
@@ -117,5 +117,5 @@
         <parent link="boat_link"/>
         <child link="motor_link"/>
-        <origin xyz="-0.91 0.0 -0.09" rpy="0 0 0"/>
+        <origin xyz="-0.905 0.0 0.115" rpy="0 0 0"/>
         <axis xyz="0 0 1"/>
         <limit effort="-1" velocity="-1" lower="-0.9" upper="0.9"/>
